File: pcb/2hu8-left/2hu8-left.kicad_sch (KiCad schematic)
At the start: 23 parts, among them U1 ProMicro, U2 TRRS, U3 TRRS

Commit message: final initial design for the boards
Parts:
- removed D10, D7, D8, D9: (no value), ScottoKeebs_Scotto:Diode_DO-35, symbol ScottoKeebs:Placeholder_Diode
- removed S10, S7, S8, S9: (no value), ScottoKeebs_MX:MX_PCB_1.00u, symbol ScottoKeebs:Placeholder_Keyswitch
- removed U3: TRRS, ScottoKeebs_Components:TRRS_PJ-320A, symbol ScottoKeebs:Placeholder_TRRS
